File: Hardware/Cerebro.sch (KiCad schematic (older format))
At the start: 2 parts, among them U1 PCB, U6 ATSAMD21G18A-AUT

Commit message: update samd21e
Parts:
- removed U6: ATSAMD21G18A-AUT, Package_QFP:TQFP-48_7x7mm_P0.5mm, symbol MCU_Microchip_SAMD:ATSAMD21G18A-AUT
- added U?: ATSAMD21E18A, Package_QFP:TQFP-32_7x7mm_P0.8mm, symbol electroniccats:ATSAMD21E18A
- U1: symbol 001-rescue:PCB-Reverse_mount_leds -> Cerebro-rescue:PCB-Reverse_mount_leds-001-rescue
Changed lines of the file:
@@
 EESchema Schematic File Version 4
-LIBS:001-cache
+LIBS:Cerebro-cache
 EELAYER 30 0
 EELAYER END
@@
 Sheet 1 1
 Title ""
-Date ""
-Rev ""
-Comp ""
-Comment1 ""
+Date "2019-10-25"
+Rev "0.1"
+Comp "Electronic Cats"
+Comment1 "Un diseño para Moon Makers"
 Comment2 ""
 Comment3 ""
-Comment4 ""
+Comment4 "Andres Sabas"
 $EndDescr
 $Comp
@@
 	10750 1250 10750 1125
 $Comp
-L wickerlib:VIN #PWR01
+L Cerebro-rescue:VIN-wickerlib #PWR01
 U 1 1 5DA054F6
 P 10750 1125
@@
 $EndComp
 $Comp
-L 001-rescue:PCB-Reverse_mount_leds U1
+L Cerebro-rescue:PCB-Reverse_mount_leds-001-rescue U1
 U 1 1 5DA40039
 P 9900 2050
@@
 PCB Art & Logos
 $Comp
-L MCU_Microchip_SAMD:ATSAMD21G18A-AUT U6
-U 1 1 5DB054F1
-P 4825 3500
-F 0 "U6" H 4825 1511 50  0000 C CNN
-F 1 "ATSAMD21G18A-AUT" H 4825 1420 50  0000 C CNN
-F 2 "Package_QFP:TQFP-48_7x7mm_P0.5mm" H 3875 1750 50  0001 C CNN
-F 3 "http://ww1.microchip.com/downloads/en/DeviceDoc/SAMD21-Family-DataSheet-DS40001882D.pdf" H 4825 4500 50  0001 C CNN
-	1    4825 3500
+L electroniccats:ATSAMD21E18A U?
+U 1 1 5DB2F8CF
+P 6755 3465
+F 0 "U?" H 7120 5319 45  0000 C CNN
+F 1 "ATSAMD21E18A" H 7120 5235 45  0000 C CNN
+F 2 "Package_QFP:TQFP-32_7x7mm_P0.8mm" H 6785 3615 20  0001 C CNN
+F 3 "https://www.mouser.mx/datasheet/2/268/SAM-D21-Family-Datasheet-DS40001882C-1381353.pdf" H 6755 3465 60  0001 C CNN
+	1    6755 3465
 	1    0    0    -1
 $EndComp

Commit message: basic componets
Parts:
- added C1: 1uF, symbol Device:CP1_Small
- added C10, C11, C6: 220nF, symbol Device:C_Small
- added C12: 25nF, symbol Device:C_Small
- added C13: 100nF, symbol Device:C_Small
- added C14, C2, C3, C8: 0.1uF, symbol Device:C_Small
- added C4: 1uF, symbol Device:C_Small
- added C5: 10nF, symbol Device:C_Small
- added C7, C9: 10uF, symbol Device:C_Small
- added D1, D2: MBR120, Package_TO_SOT_THT:TO-220-2_Vertical, symbol Diode:MBR735
- added D3, D4: LED, symbol Device:LED
- added F1: Fuse, symbol Device:Fuse
- added J1: Batt_9V, symbol Connector:Screw_Terminal_01x02
- added J2: USB_B, symbol Connector:USB_B
- added J3: Electrodos, symbol Connector:Conn_01x03_Female
- added J4: SWD, symbol Connector_Generic:Conn_02x02_Counter_Clockwise
- added R1: 1M, symbol Device:R_Small
- added R10: 560, symbol Device:R_Small
- added R11, R9: 330, symbol Device:R_Small
- added R2, R7: 100K, symbol Device:R_Small
- added R3: 220, symbol Device:R_Small
- added R4, R6: 180K, symbol Device:R_Small
- added R5: 47K, symbol Device:R_Small
- added R8: 220K, symbol Device:R_Small
- added RV1: 1K, symbol Device:R_POT_Small
- added SW1: SW_Push, symbol Switch:SW_Push
- added U1: TL084CN, symbol Amplifier_Operational:TL084CN
- added U4: AP2112K-3.3TRG1, SOT95P285X140-5N, symbol electroniccats:AP2112K-3.3TRG1
- added U5: AD620, symbol Amplifier_Instrumentation:AD620
- gave numbers to parts that had none: 1
- renumbered U1 to U2
Connections:
- net GND: now also U3.10 (GND), U3.28 (GNDA), C13.2, C14.2, C2.2, C3.2, C4.2, C7.2, C8.2, C9.2, D3.1 (K), D4.1 (K), J1.1 (Pin_1), J2.4 (GND), J2.5 (Shield), J3.3 (Pin_3), J4.4 (Pin_4), R1.1, R5.2, RV1.3, SW1.1, U1.11 (GND), U1.12 (POS4), U1.3 (POS1), U4.2 (GND), U5.4 (Vs-), U5.5 (Ref)
- net VCC: now also D2.2 (A), F1.2
- net SIGNAL: now reaches U3.11 (PA08/I2C/AIN16/SERCOM0+2.0/I2SD1)
- net SIGNAL: now also C5.1, R2.1, U1.8 (OUT3)
- net D-: now reaches U3.23 (PA24/I12/SERCOM3+5.2/D-)
- net D-: now also J2.2 (D-)
- net D+: now reaches U3.24 (PA25/I13/SERCOM3+5.3/D+)
- net D+: now also J2.3 (D+)
- net at U3.26 (/RESET): now also SW1.2
- net LED: now reaches U3.27 (PA28/I8)
- net LED: now also R11.1
- net at U3.29 (VDDCORE): now also C4.1
- net +3V3: now reaches U3.30 (VDDIN)
- net +3V3: now also U3.9 (VDDA), C2.1, C8.1, C9.1, J4.2 (Pin_2), R9.1, U4.5 (VOUT)
- net SWCLK: now reaches U3.31 (PA30/I10/SECOM1.2/SWCLK)
- net SWCLK: now also J4.3 (Pin_3)
- net SWDIO: now reaches U3.32 (PA31/I11/SECOM1.3/SWDIO)
- net SWDIO: now also J4.1 (Pin_1)
- new net: F1.1, J2.1 (VBUS)
- new net: R10.2, U5.1 (Rg)
- new net: J3.1 (Pin_1), U5.2 (-)
- new net: J3.2 (Pin_2), U5.3 (+)
- new net: C6.1, U5.6
- new net: R10.1, U5.8 (Rg)
- new net: C7.1, D1.1 (K), D2.1 (K), U4.1 (VIN)
- new net: C10.1, C11.1, C6.2, R5.1
- new net: C13.1, R4.2, R6.1, R7.2
- new net: C1.2, R1.2
- new net: R3.2, RV1.2
- new net: D3.2 (A), R9.2
- new net: D4.2 (A), R11.2
- new net +9V: C14.1, C3.1, D1.2 (A), J1.2 (Pin_2), R6.2, U1.4 (VCC), U5.7 (Vs+)
- new net NEG1: C10.2, R8.1, U1.2 (NEG1)
- new net NEG3: C5.2, R2.2, R3.1, U1.9 (NEG3)
- new net NEG4: C12.2, R7.1, U1.13 (NEG4)
- new net OUT1: C11.2, R8.2, U1.1 (OUT1)
- new net OUT4: C1.1, C12.1, R4.1, U1.14 (OUT4)
- new net POS3: U1.10 (POS3)
- no-connect marks 0 -> 24
Other:
- note added: "NOTA: AREF no lo necesitan?"
- note added: "NOTA: Potenciometro \na nada o al aire?"
- moved on the sheet: U3
